File: Hardware/CAD/Eagle files/PSU.sch (EAGLE design)
At the start: 6 parts, among them IC1 7805DT, J1 AC in

Commit message: initial release
Parts:
- removed B1: DB107S, rectifier:DBDB107G
- removed C8: 100n, rcl:C-EUC0805
- removed IC1: 7805DT, adafruit:7805DT
- added B2: RECTIFIER-2KBB, rectifier:RECTIFIER-2KBB
- added C1: 1u, adafruit:CPOL-USE2.5-5
- added IC2: 7805TV, linear:7805TV
- C6: value 1000u -> 4700u; device adafruit:CPOL-US150CLZ-1010 -> adafruit:CPOL-USE7.5-16
- C7: value 22u -> 220u; device adafruit:CPOL-US153CLV-0405 -> adafruit:CPOL-USE2.5-6
Connections:
- net GND: now also B2.-, C1.-, IC2.GND; no longer B1.-, C8.2, IC1.GND
- net N$105: now also B2.AC1; no longer B1.AC1
- net N$107: now also B2.AC2; no longer B1.AC2
- net N$108: now also B2.+, IC2.VI; no longer B1.+, IC1.VI
- net VCC: now also C1.+, IC2.VO; no longer C8.1, IC1.VO
Other:
- moved on the sheet: C6, C7, J1
