File: Hardware/CAD/Eagle files/VU-Meter.brd (EAGLE design)
At the start: 266.7 x 27 mm, 80 parts, among them IC1 7805DT, IC2 MCP6004, J1 AC in, J3 RCA, U1 ATMEGA328P_TQFP, U10 SN74HC595D, U11 SN74HC595D, U2 SN74HC595D, U3 SN74HC595D, U4 SN74HC595D, U5 SN74HC595D, U6 SN74HC595D, U7 SN74HC595D, U8 SN74HC595D, U9 SN74HC595D, Y1 16MHz

Commit message: initial release
Parts:
- removed B1: DB107S, rectifier:DB
- removed C6: 1000u, adafruit:150CLZ-1010
- removed C7: 22u, adafruit:153CLV-0405
- removed C8: 100n, rcl:C0805
- removed IC1: 7805DT, adafruit:TO252
- J1: value AC in -> PWR in (+5V)
- moved R9 21.3 mm to (4.45, 15.2)
- moved R6 21.1 mm to (4.45, 12.7)
- moved R1 21.0 mm to (31.1, 3.81)
- moved C2 21.0 mm to (38.7, 17.1)
- moved J3 20.9 mm to (3.81, 17.8)
- moved C3 20.4 mm to (36.8, 20.3)
- moved Y1 20.3 mm to (35.6, 17.1)
- moved C4 20.3 mm to (38.1, 12.7)
- moved C5 20.3 mm to (35.6, 12.7)
- moved D3 19.7 mm to (55.2, 7.62)
- moved RN2 19.7 mm to (55.2, 15.2)
- moved C1 19.7 mm to (21.0, 16.5)
- moved C15 19.7 mm to (106.0, 22.9), turned to 0 degrees
- moved D1 19.7 mm to (12.1, 15.2)
- moved D10 19.7 mm to (233.0, 7.62)
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Connections:
- removed net N$105: B1.AC1, J1.2
- removed net N$107: B1.AC2, J1.1
- removed net N$108: B1.+, C6.+, C7.+, IC1.1
- net GND: now also J1.1; no longer B1.-, C6.-, C7.-, C8.2, IC1.3
- net HC595_RCK: now also U1.11; no longer U1.2
- net HC595_SCK: now also U1.10; no longer U1.9
- net HC595_SCL: now also U1.9; no longer U1.10
- net HC595_SER: now also U1.2; no longer U1.11
- net VCC: now also J1.2; no longer C8.1, IC1.2
Routing:
- net VCC: track 0.00 -> 340.8 mm, vias 0 -> 13
- net HC595_RCK: track 0.00 -> 273.6 mm, vias 0 -> 20
- net HC595_SCK: track 0.00 -> 267.2 mm, vias 0 -> 20
- net HC595_/OE: track 0.00 -> 245.3 mm
- net HC595_SCL: track 0.00 -> 229.8 mm
- net GND: track 0.00 -> 80.2 mm, vias 0 -> 45
- net HC595_SER: track 0.00 -> 23.9 mm
- net N$4: track 0.00 -> 20.1 mm, vias 0 -> 2
- net N$2: track 0.00 -> 19.1 mm, vias 0 -> 2
- net N$1: track 0.00 -> 17.6 mm
- net RST: track 0.00 -> 17.1 mm, vias 0 -> 1
- net RCTFD_AUDIO: track 0.00 -> 17.0 mm
- net ADC: track 0.00 -> 15.1 mm, vias 0 -> 2
- net N$96: track 0.00 -> 15.0 mm
- net N$21: track 0.00 -> 15.0 mm
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- added copper zone on layer 16, net GND
Other:
- board size 266.7 x 27 mm -> 247 x 27.9 mm

Commit message: Initial release
Parts:
- removed C19, C20, C21: 100n, rcl:C0805
- removed J3: RCA, heol:1X02
- added C6, C8: 100n, rcl:C0805
- added C7: 22n, rcl:C0805
- added J2: RCA, heol:1X02
- C10: value 22n -> 100n
- D10, D3, D4, D5, D6, D7, D8, D9: device SparkFun-LED:LED_BARGRAPH_10 -> heol:LED_BARGRAPH_OFFBOARD_RIGHT_ANGLE
- moved C11 81.3 mm to (86.4, 19.1), turned to 0 degrees
- moved C12 61.7 mm to (106.7, 19.1)
- moved C15 61.7 mm to (167.6, 19.1)
- moved C16 61.1 mm to (188.0, 19.1)
- moved C17 61.1 mm to (208.3, 19.1)
- moved C18 61.1 mm to (228.6, 19.1)
- moved C13 61.1 mm to (127.0, 19.1)
- moved C14 61.1 mm to (147.3, 19.1)
- moved C10 47.5 mm to (66.0, 19.1), turned to 0 degrees
- moved C9 26.0 mm to (45.4, 19.1), turned to 0 degrees
- moved D10 12.7 mm to (221.0, 3.81), turned to 0 degrees
- moved D3 12.7 mm to (43.2, 3.81), turned to 0 degrees
- moved D4 12.7 mm to (68.6, 3.81), turned to 0 degrees
- moved D5 12.7 mm to (94.0, 3.81), turned to 0 degrees
- moved D6 12.7 mm to (119.4, 3.81), turned to 0 degrees
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- renumbered IC2 to IC1
Connections:
- net ADC: now also C6.2; no longer C9.2
- net GND: now also C7.1, C8.1, C9.1, D10.P$11, D10.P$12, D3.P$11, D3.P$12, D4.P$11, D4.P$12, D5.P$11, D5.P$12, D6.P$11, D6.P$12, D7.P$11, D7.P$12, D8.P$11, D8.P$12, D9.P$11, D9.P$12, J2.2; no longer C19.1, C20.1, C21.1, D10.11, D10.12, D10.13, D10.14, D10.15, D10.16, D10.17, D10.18, D10.19, D10.20, D3.11, D3.12, D3.13, D3.14, D3.15, D3.16, D3.17, D3.18, D3.19, D3.20, D4.11, D4.12, D4.13, D4.14, D4.15, D4.16, D4.17, D4.18, D4.19, D4.20, D5.11, D5.12, D5.13, D5.14, D5.15, D5.16, D5.17, D5.18, D5.19, D5.20, D6.11, D6.12, D6.13, D6.14, D6.15, D6.16, D6.17, D6.18, D6.19, D6.20, D7.11, D7.12, D7.13, D7.14, D7.15, D7.16, D7.17, D7.18, D7.19, D7.20, D8.11, D8.12, D8.13, D8.14, D8.15, D8.16, D8.17, D8.18, D8.19, D8.20, D9.11, D9.12, D9.13, D9.14, D9.15, D9.16, D9.17, D9.18, D9.19, D9.20, J3.2
- net N$11: now also D3.P$2; no longer D3.9
- net N$12: now also D3.P$3; no longer D3.8
- net N$13: now also D3.P$4; no longer D3.7
- net N$14: now also D3.P$5; no longer D3.6
- net N$15: now also D3.P$6; no longer D3.5
- net N$16: now also D3.P$7; no longer D3.4
- net N$17: now also D3.P$8; no longer D3.3
- net N$22: now also D3.P$9; no longer D3.2
- net N$23: now also D3.P$10; no longer D3.1
- net N$24: now also D4.P$1; no longer D4.10
- net N$25: now also D4.P$2; no longer D4.9
- net N$26: now also D4.P$3; no longer D4.8
- net N$27: now also D4.P$4; no longer D4.7
- net N$28: now also D4.P$5; no longer D4.6
- net N$29: now also D4.P$6; no longer D4.5
- net N$30: now also D4.P$7; no longer D4.4
- net N$31: now also D4.P$8; no longer D4.3
- net N$32: now also D4.P$9; no longer D4.2
- net N$33: now also D4.P$10; no longer D4.1
- net N$34: now also D5.P$1; no longer D5.10
- net N$35: now also D5.P$2; no longer D5.9
- net N$36: now also D5.P$3; no longer D5.8
- net N$37: now also D5.P$4; no longer D5.7
- net N$38: now also D5.P$5; no longer D5.6
- net N$39: now also D5.P$6; no longer D5.5
- net N$40: now also D5.P$7; no longer D5.4
- net N$41: now also D5.P$8; no longer D5.3
- net N$42: now also D5.P$9; no longer D5.2
- net N$43: now also D5.P$10; no longer D5.1
- net N$44: now also D6.P$1; no longer D6.10
- net N$45: now also D6.P$2; no longer D6.9
- net N$46: now also D6.P$3; no longer D6.8
- net N$47: now also D6.P$4; no longer D6.7
- net N$48: now also D6.P$5; no longer D6.6
- net N$49: now also D6.P$6; no longer D6.5
- net N$50: now also D6.P$7; no longer D6.4
- net N$51: now also D6.P$8; no longer D6.3
- net N$52: now also D6.P$9; no longer D6.2
- net N$53: now also D6.P$10; no longer D6.1
- net N$54: now also D7.P$1; no longer D7.10
- net N$55: now also D7.P$2; no longer D7.9
- net N$56: now also D7.P$3; no longer D7.8
- net N$57: now also D7.P$4; no longer D7.7
- net N$58: now also D7.P$5; no longer D7.6
- net N$59: now also D7.P$6; no longer D7.5
- net N$6: now also J2.1; no longer J3.1
- net N$60: now also D7.P$7; no longer D7.4
- net N$61: now also D7.P$8; no longer D7.3
- net N$62: now also D7.P$9; no longer D7.2
- net N$63: now also D7.P$10; no longer D7.1
- net N$64: now also D8.P$1; no longer D8.10
- net N$65: now also D8.P$2; no longer D8.9
- net N$66: now also D8.P$3; no longer D8.8
- net N$67: now also D8.P$4; no longer D8.7
- net N$68: now also D8.P$5; no longer D8.6
- net N$69: now also D8.P$6; no longer D8.5
- net N$7: now also C6.1; no longer C9.1
- net N$70: now also D8.P$7; no longer D8.4
- net N$71: now also D8.P$8; no longer D8.3
- net N$72: now also D8.P$9; no longer D8.2
- net N$73: now also D8.P$10; no longer D8.1
- net N$74: now also D9.P$1; no longer D9.10
- net N$75: now also D9.P$2; no longer D9.9
- net N$76: now also D9.P$3; no longer D9.8
- net N$77: now also D9.P$4; no longer D9.7
- net N$78: now also D9.P$5; no longer D9.6
- net N$79: now also D9.P$6; no longer D9.5
- net N$8: now also C7.2; no longer C10.2
- net N$80: now also D9.P$7; no longer D9.4
- net N$81: now also D9.P$8; no longer D9.3
- net N$82: now also D9.P$9; no longer D9.2
- net N$83: now also D9.P$10; no longer D9.1
- net N$84: now also D10.P$1; no longer D10.10
- net N$85: now also D10.P$2; no longer D10.9
- net N$86: now also D10.P$3; no longer D10.8
- net N$87: now also D10.P$4; no longer D10.7
- net N$88: now also D10.P$5; no longer D10.6
- net N$89: now also D10.P$6; no longer D10.5
- net N$9: now also D3.P$1; no longer D3.10
- net N$90: now also D10.P$7; no longer D10.4
- net N$91: now also D10.P$8; no longer D10.3
- net N$92: now also D10.P$9; no longer D10.2
- net N$93: now also D10.P$10; no longer D10.1
- net VCC: now also C10.2, C8.2, C9.2; no longer C19.2, C20.2, C21.2
Routing:
- net VCC: track 340.8 -> 324.5 mm, vias 13 -> 15
- net N$22: track 6.47 -> 11.8 mm
- net N$23: track 4.80 -> 10.2 mm
- net HC595_RCK: track 273.6 -> 268.4 mm
- net HC595_SCK: track 267.2 -> 262.1 mm
- net HC595_SCL: track 229.8 -> 224.9 mm
- net N$63: track 4.80 -> 9.60 mm
- net N$62: track 6.47 -> 11.1 mm
- net N$73: track 3.21 -> 7.81 mm
- net N$33: track 3.21 -> 7.81 mm
- net N$74: track 3.21 -> 7.76 mm
- net N$34: track 3.21 -> 7.76 mm
- net HC595_/OE: track 245.3 -> 241.2 mm
- net HC595_SER: track 23.9 -> 19.7 mm
- net N$88: track 3.88 -> 7.95 mm
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Other:
- board size 247 x 27.9 mm -> 247 x 24.1 mm
- board text added: "-+"
- board text added: "VU-meter Heol Fief 2019"

Commit message: Initial release
Parts:
- moved C2 1.80 mm to (41.0, 15.9), turned to 180 degrees
- moved C3 1.00 mm to (41.0, 18.1), turned to 180 degrees
Routing:
- net GND: track 77.7 -> 65.3 mm, vias 45 -> 47
- net N$99: track 7.70 -> 5.43 mm
- net N$100: track 8.17 -> 9.35 mm
- added copper zone on layer 1, net GND
Other:
- board size 247 x 24.1 mm -> 252.7 x 24.1 mm

Commit message: Initial release
Parts:
- added J3: UART_DBG, SparkFun-Connectors:1X02
- moved R1 1.27 mm to (31.1, 2.54)
- moved R2 1.27 mm to (39.4, 2.54)
Connections:
- new net N$103: J3.2, U1.30
- new net N$104: J3.1, U1.31
Routing:
- net N$103: track 0.00 -> 9.54 mm
- net N$104: track 0.00 -> 5.36 mm
- net GAIN: track 6.18 -> 7.45 mm
- net VCC: track 324.5 -> 325.0 mm
- net THRESHOLD: track 10.8 -> 11.4 mm
Other:
- board text added: "RX"
- board text added: "TX"
Changed lines of the file:
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@@
 <hole x="247.65" y="2.54" drill="3"/>
 <hole x="123.825" y="12.065" drill="3"/>
+<text x="40.64" y="6.0325" size="1.27" layer="25" font="vector" ratio="15" rot="R180">RX</text>
+<text x="37.7825" y="6.0325" size="1.27" layer="25" font="vector" ratio="15" rot="R180">TX</text>
 </plain>
 <attributes>
@@
 <attribute name="VALUE" x="2.54" y="18.288" size="1.27" layer="27" font="vector" ratio="31"/>
 </element>
-<element name="R1" library="heol" package="1X03" value="10k" x="31.115" y="3.81" smashed="yes" rot="R180">
-<attribute name="NAME" x="29.5275" y="2.413" size="1.27" layer="25" font="vector" ratio="15" rot="R180"/>
-<attribute name="VALUE" x="32.385" y="5.842" size="1.27" layer="27" font="vector" ratio="31" rot="R180"/>
+<element name="R1" library="heol" package="1X03" value="10k" x="31.115" y="2.54" smashed="yes" rot="R180">
+<attribute name="NAME" x="30.1625" y="4.2545" size="1.27" layer="25" font="vector" ratio="15"/>
+<attribute name="VALUE" x="32.385" y="4.572" size="1.27" layer="27" font="vector" ratio="31" rot="R180"/>
 </element>
 <element name="R10" library="resistor" library_urn="urn:adsk.eagle:library:348" package="R0805" package3d_urn="urn:adsk.eagle:package:23553/2" value="100k" x="19.685" y="9.525" smashed="yes" rot="R180">
@@
 <attribute name="VALUE" x="19.685" y="12.3825" size="1.27" layer="27" rot="R90"/>
 </element>
-<element name="R2" library="heol" package="1X03" value="10k" x="39.37" y="3.81" smashed="yes" rot="R180">
-<attribute name="NAME" x="37.7825" y="2.413" size="1.27" layer="25" font="vector" ratio="15" rot="R180"/>
-<attribute name="VALUE" x="40.64" y="5.842" size="1.27" layer="27" font="vector" ratio="31" rot="R180"/>
+<element name="R2" library="heol" package="1X03" value="10k" x="39.37" y="2.54" smashed="yes" rot="R180">
+<attribute name="NAME" x="33.3375" y="4.2545" size="1.27" layer="25" font="vector" ratio="15"/>
+<attribute name="VALUE" x="40.64" y="4.572" size="1.27" layer="27" font="vector" ratio="31" rot="R180"/>
 </element>
 <element name="R3" library="resistor" library_urn="urn:adsk.eagle:library:348" package="R0805" package3d_urn="urn:adsk.eagle:package:23553/2" value="100k" x="17.145" y="17.78" smashed="yes" rot="R90">
@@
 </element>
 <element name="U1" library="SparkFun-IC-Microcontroller" library_urn="urn:adsk.eagle:library:525" package="TQFP32-08" package3d_urn="urn:adsk.eagle:package:38945/1" value="ATMEGA328P_TQFP" x="31.115" y="12.065" smashed="yes" rot="R180">
-<attribute name="NAME" x="35.8775" y="7.9375" size="1.27" layer="25" font="vector" ratio="15" rot="R180" align="bottom-center"/>
+<attribute name="NAME" x="26.9875" y="7.9375" size="1.27" layer="25" font="vector" ratio="15" rot="R180" align="bottom-center"/>
 <attribute name="PROD_ID" value="IC-09069" x="13.335" y="61.595" size="1.778" layer="27" rot="R180" display="off"/>
 <attribute name="VALUE" x="31.115" y="18.415" size="1.27" layer="27" font="vector" ratio="31" rot="R180" align="bottom-center"/>
@@
 <attribute name="NAME" x="222.5675" y="5.715" size="1.27" layer="21" font="vector" ratio="15"/>
 <attribute name="VALUE" x="230.1875" y="5.715" size="1.27" layer="21" font="vector" ratio="15"/>
+</element>
+<element name="J3" library="SparkFun-Connectors" library_urn="urn:adsk.eagle:library:513" package="1X02" package3d_urn="urn:adsk.eagle:package:38039/1" value="UART_DBG" x="37.1475" y="7.62" smashed="yes">
+<attribute name="NAME" x="40.64" y="8.382" size="1.27" layer="25" font="vector" ratio="15"/>
+<attribute name="VALUE" x="35.8775" y="5.588" size="0.6096" layer="27" font="vector" ratio="20"/>
 </element>
 </elements>
@@
 <wire x1="36.43" y1="11.665" x2="36.83" y2="12.065" width="0.254" layer="1"/>
 <wire x1="36.83" y1="12.065" x2="36.83" y2="13.335" width="0.254" layer="1"/>
-<wire x1="31.115" y1="3.81" x2="33.02" y2="1.905" width="0.254" layer="1"/>
-<wire x1="33.02" y1="1.905" x2="38.1" y2="1.905" width="0.254" layer="1"/>
-<wire x1="38.1" y1="1.905" x2="39.37" y2="3.175" width="0.254" layer="1"/>
-<wire x1="39.37" y1="3.175" x2="39.37" y2="3.81" width="0.254" layer="1"/>
-<wire x1="31.115" y1="3.81" x2="31.115" y2="6.0325" width="0.254" layer="16"/>
+<wire x1="31.115" y1="2.54" x2="32.385" y2="1.27" width="0.254" layer="1"/>
+<wire x1="32.385" y1="1.27" x2="38.4175" y2="1.27" width="0.254" layer="1"/>
+<wire x1="39.37" y1="2.54" x2="39.37" y2="2.2225" width="0.254" layer="1"/>
+<wire x1="39.37" y1="2.2225" x2="38.4175" y2="1.27" width="0.254" layer="1"/>
+<wire x1="31.115" y1="2.54" x2="31.115" y2="6.0325" width="0.254" layer="16"/>
 <wire x1="31.115" y1="6.0325" x2="33.655" y2="8.5725" width="0.254" layer="16"/>
 <wire x1="33.655" y1="8.5725" x2="33.655" y2="11.43" width="0.254" layer="16"/>
@@
 <contactref element="U1" pad="24"/>
 <contactref element="R1" pad="2"/>
-<wire x1="26.8224" y1="9.265" x2="26.8224" y2="5.5626" width="0.1778" layer="1"/>
-<wire x1="26.8224" y1="5.5626" x2="28.575" y2="3.81" width="0.1778" layer="1"/>
+<wire x1="26.8224" y1="9.265" x2="26.8224" y2="4.2926" width="0.1778" layer="1"/>
+<wire x1="26.8224" y1="4.2926" x2="28.575" y2="2.54" width="0.1778" layer="1"/>
 </signal>
 <signal name="THRESHOLD">
@@
 <wire x1="28.315" y1="7.7724" x2="28.315" y2="6.61" width="0.1778" layer="1"/>
 <wire x1="28.315" y1="6.61" x2="28.575" y2="6.35" width="0.1778" layer="1"/>
-<wire x1="28.575" y1="6.35" x2="34.29" y2="6.35" width="0.1778" layer="1"/>
-<wire x1="34.29" y1="6.35" x2="36.83" y2="3.81" width="0.1778" layer="1"/>
+<wire x1="28.575" y1="6.35" x2="33.02" y2="6.35" width="0.1778" layer="1"/>
+<wire x1="33.02" y1="6.35" x2="36.83" y2="2.54" width="0.1778" layer="1"/>
 </signal>
 <signal name="N$1">
@@
 <wire x1="239.325" y1="8.325" x2="239.325" y2="10.805" width="0.1778" layer="1"/>
 </signal>
+<signal name="N$103">
+<contactref element="U1" pad="30"/>
+<contactref element="J3" pad="2"/>
+<wire x1="32.315" y1="7.7724" x2="32.315" y2="7.055" width="0.1778" layer="1"/>
+<wire x1="32.315" y1="7.055" x2="32.6898" y2="6.6802" width="0.1778" layer="1"/>
+<wire x1="36.344475" y1="6.0325" x2="38.735" y2="6.0325" width="0.1778" layer="1"/>
+<wire x1="35.696775" y1="6.6802" x2="36.344475" y2="6.0325" width="0.1778" layer="1"/>
+<wire x1="32.6898" y1="6.6802" x2="35.696775" y2="6.6802" width="0.1778" layer="1"/>
+<wire x1="38.735" y1="6.0325" x2="39.6875" y2="6.985" width="0.1778" layer="1"/>
+<wire x1="39.6875" y1="6.985" x2="39.6875" y2="7.62" width="0.1778" layer="1"/>
+</signal>
+<signal name="N$104">
+<contactref element="U1" pad="31"/>
+<contactref element="J3" pad="1"/>
+<wire x1="33.115" y1="7.7724" x2="33.115" y2="8.35" width="0.1778" layer="1"/>
+<wire x1="33.115" y1="8.35" x2="33.655" y2="8.89" width="0.1778" layer="1"/>
+<wire x1="33.655" y1="8.89" x2="34.29" y2="8.89" width="0.1778" layer="1"/>
+<wire x1="34.29" y1="8.89" x2="35.56" y2="7.62" width="0.1778" layer="1"/>
+<wire x1="35.56" y1="7.62" x2="37.1475" y2="7.62" width="0.1778" layer="1"/>
+</signal>
 </signals>

Commit message: Initial release
Initial release

Initial release

Initial release

Create Enclosure Mechanical Drawing.pdf

Add pcb prictures

Update README.md

Update README.md

Update README.md

Add .gitignore

Initial release

Initial release
Parts:
- added J4: GPIO, SparkFun-Connectors:1X04
- moved R11 0.64 mm to (17.8, 13.0)
- moved Y1 0.32 mm to (37.1, 17.5)
Connections:
- new net N$105: J4.4, U1.12
- new net N$106: J4.3, U1.13
- new net N$107: J4.2, U1.14
- net GND: now also J4.1
Routing:
- net N$105: track 0.00 -> 5.99 mm
- net N$107: track 0.00 -> 5.92 mm
- net N$106: track 0.00 -> 5.27 mm
- net HC595_SCL: track 224.9 -> 223.8 mm
- net HC595_RCK: track 268.4 -> 267.2 mm
- net HC595_SCK: track 262.1 -> 261.0 mm
- net VCC: track 325.0 -> 324.1 mm
- net N$99: track 5.43 -> 6.06 mm
Other:
- board text added: "Heol Fief 2019"
- board text added: "VU-meter"
- board text removed: "VU-meter Heol Fief 2019"
