File: Hardware/CAD/Eagle files/VU-Meter.sch (EAGLE design)
At the start: 65 parts, among them IC1 MCP6004, IC3 7805DT, J1 RCA, J3 AC in, U1 ATMEGA328P_TQFP, U10 SN74HC595D, U11 SN74HC595D, U2 SN74HC595D, U3 SN74HC595D, U4 SN74HC595D, U5 SN74HC595D, U6 SN74HC595D, U7 SN74HC595D, U8 SN74HC595D, U9 SN74HC595D, Y1 16MHz

Commit message: initial release
Parts:
- added R10, R11: 10k, heol:POT_OFFBOARD
Connections:
- new net GAIN: R10.S, U1.PC1(ADC1)
- new net THRESHOLD: R11.S, U1.PC2(ADC2)
- net GND: now also R10.A, R11.A
- net VCC: now also R10.E, R11.E

Commit message: initial release
Parts:
- removed IC3: 7805DT, adafruit:7805DT
- added C12, C13, C14, C15, C16, C17, C18, C19, C20, C21, C8: 100n, rcl:C-EUC0805
- added C6: 1000u, adafruit:CPOL-US150CLZ-1010
- added C7: 22u, adafruit:CPOL-US153CLV-0405
- added IC2: MCP6004, adafruit:QUAD_OPAMPD
- C10: value 22u -> 22n; device adafruit:CPOL-US153CLV-0405 -> rcl:C-EUC0805
- C5: value 22n -> 100n
- C9: value 1000u -> 100n; device adafruit:CPOL-US150CLZ-1010 -> rcl:C-EUC0805
- IC1: value MCP6004 -> 7805DT; device adafruit:QUAD_OPAMPD -> adafruit:7805DT
- J1: value RCA -> AC in; device SparkFun-Connectors:RCA -> SparkFun-Connectors:CONN_02
- J3: value AC in -> RCA; device SparkFun-Connectors:CONN_02 -> heol:MONO_JACK_OFFBOARD
- R1, R2: value 100k -> 10k; device resistor:R-EU_R0805 -> heol:POT_OFFBOARD
- R10, R11: value 10k -> 100k; device heol:POT_OFFBOARD -> resistor:R-EU_R0805
- R5: value 47k -> 100k
- R6: value 24k -> 100k
- R7: value 100k -> 47k
- R8: value 100k -> 24k
- RN1, RN10, RN11, RN12, RN13, RN14, RN15, RN16, RN17, RN18, RN19, RN2, RN20, RN3, RN4, RN5, RN6, RN7, RN8, RN9: value (none) -> 820
Connections:
- net ADC: now also C9.2, IC2C.-IN, IC2C.OUT; no longer C4.2, IC1C.-IN, IC1C.OUT
- net GAIN: now also R1.S; no longer R10.S
- net GND: now also C10.1, C11.1, C12.1, C13.1, C14.1, C15.1, C16.1, C17.1, C18.1, C19.1, C20.1, C21.1, C4.2, C5.2, C6.-, C7.-, C8.2, IC1.GND, IC2A.+IN, IC2P.V-, J3.SLEEVE, R1.A, R11.2, R2.A; no longer C10.-, C11.2, C5.1, C9.-, IC1A.+IN, IC1P.V-, IC3.GND, J1.PIN, R10.A, R11.A, R9.2
- net N$1: now also IC2A.-IN, R3.1, R6.2, R9.1; no longer IC1A.-IN, R1.1, R4.2, R7.1
- net N$101: now also IC2D.-IN, IC2D.OUT; no longer IC1D.-IN, IC1D.OUT
- net N$102: now also IC2D.+IN, R10.1, R11.1; no longer IC1D.+IN, R8.1, R9.1
- net N$105: now also J1.2; no longer J3.2
- net N$107: now also J1.1; no longer J3.1
- net N$108: now also C6.+, C7.+, IC1.VI; no longer C10.+, C9.+, IC3.VI
- net N$2: now also IC2B.+IN, R9.2; no longer IC1B.+IN, R7.2
- net N$3: now also IC2A.OUT; no longer IC1A.OUT
- net N$4: now also R3.2, R4.1; no longer R1.2, R2.1
- net N$5: now also IC2B.-IN, R4.2, R5.1; no longer IC1B.-IN, R2.2, R3.1
- net N$6: now also J3.TIP, R6.1; no longer J1.SHELL, R4.1
- net N$7: now also C9.1, R7.2, R8.1; no longer C4.1, R5.2, R6.1
- net N$8: now also C10.2, IC2C.+IN, R8.2; no longer C5.2, IC1C.+IN, R6.2
- net RCTFD_AUDIO: now also IC2B.OUT, R5.2, R7.1; no longer IC1B.OUT, R3.2, R5.1
- net THRESHOLD: now also R2.S; no longer R11.S
- net VCC: now also C11.2, C12.2, C13.2, C14.2, C15.2, C16.2, C17.2, C18.2, C19.2, C20.2, C21.2, C4.1, C5.1, C8.1, IC1.VO, IC2P.V+, R1.E, R10.2, R2.E; no longer C11.1, IC1P.V+, IC3.VO, R10.E, R11.E, R8.2
Other:
- note added: "Resistor Arrays values :"

Commit message: initial release
Parts:
- removed B1: DB107S, rectifier:DBDB107G
- removed C6: 1000u, adafruit:CPOL-US150CLZ-1010
- removed C7: 22u, adafruit:CPOL-US153CLV-0405
- removed C8: 100n, rcl:C-EUC0805
- removed IC1: 7805DT, adafruit:7805DT
- J1: value AC in -> PWR in (+5V)
Connections:
- removed net N$105: B1.AC1, J1.2
- removed net N$107: B1.AC2, J1.1
- removed net N$108: B1.+, C6.+, C7.+, IC1.VI
- net GND: now also J1.1; no longer B1.-, C6.-, C7.-, C8.2, IC1.GND
- net HC595_RCK: now also U1.PD7(AIN1); no longer U1.PD4(XCK/T0)
- net HC595_SCK: now also U1.PD6(AIN0); no longer U1.PD5(T1)
- net HC595_SCL: now also U1.PD5(T1); no longer U1.PD6(AIN0)
- net HC595_SER: now also U1.PD4(XCK/T0); no longer U1.PD7(AIN1)
- net VCC: now also J1.2; no longer C8.1, IC1.VO
Other:
- moved on the sheet: J1

Commit message: Initial release
Parts:
- removed C19, C20, C21: 100n, rcl:C-EUC0805
- added C6, C8: 100n, rcl:C-EUC0805
- added C7: 22n, rcl:C-EUC0805
- C10: value 22n -> 100n
- D10: device SparkFun-LED:LED_BARGRAPH_10RED -> heol:LED_BARGRAPH_OFFBOARDLED_BARGRAPH_OFFBOARD
- D3, D4, D5, D6, D7, D8, D9: device SparkFun-LED:LED_BARGRAPH_10GREEN -> heol:LED_BARGRAPH_OFFBOARDLED_BARGRAPH_OFFBOARD
- renumbered IC2 to IC1, J3 to J2
Connections:
- net ADC: now also C6.2; no longer C9.2
- net GND: now also C7.1, C8.1, C9.1; no longer C19.1, C20.1, C21.1, D10.C2, D10.C3, D10.C4, D10.C5, D10.C6, D10.C7, D10.C8, D10.C9, D3.C2, D3.C3, D3.C4, D3.C5, D3.C6, D3.C7, D3.C8, D3.C9, D4.C2, D4.C3, D4.C4, D4.C5, D4.C6, D4.C7, D4.C8, D4.C9, D5.C2, D5.C3, D5.C4, D5.C5, D5.C6, D5.C7, D5.C8, D5.C9, D6.C2, D6.C3, D6.C4, D6.C5, D6.C6, D6.C7, D6.C8, D6.C9, D7.C2, D7.C3, D7.C4, D7.C5, D7.C6, D7.C7, D7.C8, D7.C9, D8.C2, D8.C3, D8.C4, D8.C5, D8.C6, D8.C7, D8.C8, D8.C9, D9.C2, D9.C3, D9.C4, D9.C5, D9.C6, D9.C7, D9.C8, D9.C9
- net N$7: now also C6.1; no longer C9.1
- net N$8: now also C7.2; no longer C10.2
- net VCC: now also C10.2, C8.2, C9.2; no longer C19.2, C20.2, C21.2
Other:
- moved on the sheet: C12, C13, C14, C15, C16, C17, C18

Commit message: Initial release
Parts:
- added J3: UART_DBG, SparkFun-Connectors:CONN_02
Connections:
- new net N$103: J3.2, U1.PD0(RXD)
- new net N$104: J3.1, U1.PD1(TXD)
Changed lines of the file:
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@@
 <part name="D9" library="heol" deviceset="LED_BARGRAPH_OFFBOARD" device="LED_BARGRAPH_OFFBOARD" value="GREEN"/>
 <part name="D10" library="heol" deviceset="LED_BARGRAPH_OFFBOARD" device="LED_BARGRAPH_OFFBOARD" value="RED"/>
+<part name="J3" library="SparkFun-Connectors" library_urn="urn:adsk.eagle:library:513" deviceset="CONN_02" device="" package3d_urn="urn:adsk.eagle:package:38039/1" value="UART_DBG"/>
 </parts>
 <sheets>
@@
 <instance part="P+5" gate="VCC" x="96.52" y="106.68" smashed="yes">
 <attribute name="VALUE" x="99.822" y="104.14" size="1.778" layer="96" rot="R90"/>
+</instance>
+<instance part="J3" gate="G$1" x="165.1" y="124.46" smashed="yes" rot="MR0">
+<attribute name="VALUE" x="167.64" y="119.634" size="1.778" layer="96" font="vector" rot="MR0"/>
+<attribute name="NAME" x="167.64" y="130.048" size="1.778" layer="95" font="vector" rot="MR0"/>
 </instance>
 </instances>
@@
 </segment>
 </net>
+<net name="N$103" class="0">
+<segment>
+<pinref part="U1" gate="U$1" pin="PD0(RXD)"/>
+<wire x1="147.32" y1="119.38" x2="152.4" y2="119.38" width="0.1524" layer="91"/>
+<wire x1="152.4" y1="119.38" x2="152.4" y2="127" width="0.1524" layer="91"/>
+<pinref part="J3" gate="G$1" pin="2"/>
+<wire x1="152.4" y1="127" x2="157.48" y2="127" width="0.1524" layer="91"/>
+</segment>
+</net>
+<net name="N$104" class="0">
+<segment>
+<pinref part="U1" gate="U$1" pin="PD1(TXD)"/>
+<wire x1="147.32" y1="116.84" x2="154.94" y2="116.84" width="0.1524" layer="91"/>
+<wire x1="154.94" y1="116.84" x2="154.94" y2="124.46" width="0.1524" layer="91"/>
+<pinref part="J3" gate="G$1" pin="1"/>
+<wire x1="154.94" y1="124.46" x2="157.48" y2="124.46" width="0.1524" layer="91"/>
+</segment>
+</net>

Commit message: Initial release
Initial release

Initial release

Initial release

Create Enclosure Mechanical Drawing.pdf

Add pcb prictures

Update README.md

Update README.md

Update README.md

Add .gitignore

Initial release

Initial release
Parts:
- added J4: GPIO, SparkFun-Connectors:CONN_04
Connections:
- new net N$105: J4.4, U1.PB0(ICP)
- new net N$106: J4.3, U1.PB1(OC1A)
- new net N$107: J4.2, U1.PB2(SS/OC1B)
- net GND: now also J4.1
Changed lines of the file:
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@@
 <?xml version="1.0" encoding="utf-8"?>
 <!DOCTYPE eagle SYSTEM "eagle.dtd">
-<eagle version="9.2.2">
+<eagle version="9.3.0">
 <drawing>
 <settings>
@@
 <part name="D10" library="heol" deviceset="LED_BARGRAPH_OFFBOARD" device="LED_BARGRAPH_OFFBOARD" value="RED"/>
 <part name="J3" library="SparkFun-Connectors" library_urn="urn:adsk.eagle:library:513" deviceset="CONN_02" device="" package3d_urn="urn:adsk.eagle:package:38039/1" value="UART_DBG"/>
+<part name="J4" library="SparkFun-Connectors" library_urn="urn:adsk.eagle:library:513" deviceset="CONN_04" device="" package3d_urn="urn:adsk.eagle:package:38085/1" value="GPIO"/>
+<part name="GND33" library="supply1" library_urn="urn:adsk.eagle:library:371" deviceset="GND" device=""/>
 </parts>
 <sheets>
@@
 <attribute name="NAME" x="167.64" y="130.048" size="1.778" layer="95" font="vector" rot="MR0"/>
 </instance>
+<instance part="J4" gate="G$1" x="187.96" y="91.44" smashed="yes" rot="MR0">
+<attribute name="VALUE" x="193.04" y="84.074" size="1.778" layer="96" font="vector" rot="MR0"/>
+<attribute name="NAME" x="193.04" y="99.568" size="1.778" layer="95" font="vector" rot="MR0"/>
+</instance>
+<instance part="GND33" gate="1" x="182.88" y="86.36" smashed="yes">
+<attribute name="VALUE" x="180.34" y="83.82" size="1.778" layer="96"/>
+</instance>
 </instances>
 <busses>
@@
 <wire x1="68.58" y1="71.12" x2="157.48" y2="71.12" width="0.762" layer="92"/>
 <wire x1="157.48" y1="71.12" x2="162.56" y2="76.2" width="0.762" layer="92"/>
-<wire x1="162.56" y1="91.44" x2="162.56" y2="76.2" width="0.762" layer="92"/>
+<wire x1="162.56" y1="88.9" x2="162.56" y2="76.2" width="0.762" layer="92"/>
 <label x="165.1" y="88.9" size="1.778" layer="95" rot="R270"/>
 </segment>
@@
 <bus name="SHIFT_REG_BUS:GND,HC595_/OE,HC595_RCK,HC595_SCK,HC595_SCL,HC595_SER,VCC">
 <segment>
-<wire x1="167.64" y1="116.84" x2="167.64" y2="96.52" width="0.762" layer="92"/>
+<wire x1="167.64" y1="116.84" x2="167.64" y2="99.06" width="0.762" layer="92"/>
 <label x="172.72" y="101.6" size="1.778" layer="95" rot="R90"/>
 </segment>
@@
 <pinref part="GND1" gate="1" pin="GND"/>
 </segment>
+<segment>
+<pinref part="J4" gate="G$1" pin="1"/>
+<pinref part="GND33" gate="1" pin="GND"/>
+</segment>
 </net>
 <net name="N$10" class="0">
@@
 </segment>
 </net>
+<net name="N$105" class="0">
+<segment>
+<pinref part="U1" gate="U$1" pin="PB0(ICP)"/>
+<wire x1="147.32" y1="96.52" x2="149.86" y2="96.52" width="0.1524" layer="91"/>
+<wire x1="149.86" y1="96.52" x2="182.88" y2="96.52" width="0.1524" layer="91"/>
+<pinref part="J4" gate="G$1" pin="4"/>
+</segment>
+</net>
+<net name="N$106" class="0">
+<segment>
+<pinref part="U1" gate="U$1" pin="PB1(OC1A)"/>
+<wire x1="147.32" y1="93.98" x2="149.86" y2="93.98" width="0.1524" layer="91"/>
+<wire x1="149.86" y1="93.98" x2="182.88" y2="93.98" width="0.1524" layer="91"/>
+<pinref part="J4" gate="G$1" pin="3"/>
+</segment>
+</net>
+<net name="N$107" class="0">
+<segment>
+<pinref part="U1" gate="U$1" pin="PB2(SS/OC1B)"/>
+<wire x1="147.32" y1="91.44" x2="149.86" y2="91.44" width="0.1524" layer="91"/>
+<wire x1="149.86" y1="91.44" x2="182.88" y2="91.44" width="0.1524" layer="91"/>
+<pinref part="J4" gate="G$1" pin="2"/>
+</segment>
+</net>
